Commit message: add initial service support

File: urdf/blue-slam.urdf (robot description, URDF)
Before this commit: robot blue-slam, 36 links, 35 joints
Links:
- removed link angle_bracket_plate_1
- removed link angle_bracket_plate_2
- removed link back_left_standoff
- removed link back_right_standoff
- removed link battery
- removed link camera_board
- removed link camera_lense
- removed link camera_mount_bracket_1
- removed link camera_mount_bracket_2
- removed link castor
- removed link castor_bracket
- removed link castor_wheel
- removed link compute_complex
- removed link front_base_plate
- removed link front_left_standoff
- removed link front_right_standoff
- removed link imu
- removed link imu_left_standoff
- removed link imu_right_standoff
- removed link leddar_lens
- removed link leddar_sensor
- removed link left_motor
- removed link left_motor_bracket
- removed link left_motor_output_shaft
- removed link left_motor_shaft_connector
- removed link left_wheel
- removed link right_motor
- removed link right_motor_bracket
- removed link right_motor_output_shaft
- removed link right_motor_shaft_connector
- removed link right_wheel
- removed link tail_base_plate
- removed link tail_link
- added link angle_bracket_plate_1_link; visual box size=0.026 0.024 0.002
- added link angle_bracket_plate_2_link; visual box size=0.002 0.024 0.024
- added link back_left_standoff_link; visual cylinder length=.050 radius=0.0025
- added link back_right_standoff_link; visual cylinder length=.050 radius=0.0025
- added link battery_link; visual box size=0.075 0.032 0.032
- added link bottom_tail_link; visual box size=0.144 0.024 0.008
- added link camera_board_link; visual box size=0.001 0.025 0.024
- added link camera_lens_link; visual cylinder length=0.017 radius=0.007
- added link camera_mount_bracket_1_link; visual box size=0.024 0.040 0.003
- added link camera_mount_bracket_2_link; visual box size=0.003 0.035 0.028
- added link castor_bracket_link; visual box size=0.032 0.024 0.010
- added link castor_link; visual box size=0.0305 0.025 0.026
- added link castor_wheel_link; visual cylinder length=0.012 radius=0.0125
- added link front_base_plate_link; visual box size=0.003 0.104 0.090
- added link front_left_standoff_link; visual cylinder length=.050 radius=0.0025
- added link front_right_standoff_link; visual cylinder length=.050 radius=0.0025
- added link imu_left_standoff_link; visual cylinder length=0.020 radius=.0025
- added link imu_link; visual box size=0.0267 0.0203 0.002
- added link imu_right_standoff_link; visual cylinder length=0.020 radius=.0025
- added link leddar_lens_link; visual cylinder length=0.036 radius=0.0155
- added link leddar_sensor_link; visual box size=0.0329 0.076 0.114
- added link left_motor_bracket_link; visual box size=0.037 0.003 0.037
- added link left_motor_link; visual cylinder length=0.0635 radius=0.0125
- added link left_motor_output_shaft_link; visual cylinder length=0.0125 radius=0.004
- added link left_wheel_connector_link; visual cylinder length=0.005 radius=0.011
- added link left_wheel_link; visual cylinder length=0.008 radius=0.03525
- added link raspberry_pi_link; visual box size=0.056 0.085 0.033
- added link right_motor_bracket_link; visual box size=0.037 0.003 0.037
- added link right_motor_link; visual cylinder length=0.0635 radius=0.0125
- added link right_motor_output_shaft_link; visual cylinder length=0.0125 radius=0.004
- added link right_wheel_connector_link; visual cylinder length=0.005 radius=0.011
- added link right_wheel_link; visual cylinder length=0.008 radius=0.03525
- added link tail_base_plate_link; visual box size=0.090 0.104 0.003
- link base_link: geometry visual box size=0.024 0.144 0.008
Joints:
- removed joint angle_brack_to_front_base_plate_joint
- removed joint back_left_standoff_joint
- removed joint back_right_standoff_joint
- removed joint battery_to_tail_joint
- removed joint bracket_to_left_motor_joint
- removed joint bracket_to_right_motor_joint
- removed joint camera_board_to_lense_joint
- removed joint camera_to_bracket_joint
- removed joint castor_wheel_joint
- removed joint compute_to_tail_base_plate
- removed joint front_left_standoff_joint
- removed joint front_right_standoff_joint
- removed joint imu_left_standoff_joint
- removed joint imu_right_standoff_joint
- removed joint leddar_laser_to_front_base_plate_joint
- removed joint leddar_sensor_to_lens_joint
- removed joint left_motor_joint
- removed joint left_motor_shaft_connector_joint
- removed joint left_wheel_connector_joint
- removed joint right_motor_joint
- removed joint right_motor_shaft_connector_joint
- removed joint right_wheel_connector_joint
- removed joint tail_base_plate_joint
- removed joint tail_to_angle_bracket_joint
- removed joint tail_to_tail_bracket_joint
- removed joint top_tail_link_joint
- added joint angle_bracket_to_front_base_plate_joint: type fixed, parent angle_bracket_plate_2_link, child front_base_plate_link, origin xyz=0.0025 0.0 0.032 rpy=0.0 0.0 0.0
- added joint battery_to_bottom_tail_joint: type fixed, parent bottom_tail_link, child battery_link, origin xyz=0.0 0.0 0.020 rpy=0.0 0.0 0.0
- added joint bottom_tail_to_angle_bracket_joint: type fixed, parent bottom_tail_link, child angle_bracket_plate_1_link, origin xyz=0.067 0.0 0.005 rpy=0.0 0.0 0.0
- added joint bottom_tail_to_back_left_standoff_joint: type fixed, parent bottom_tail_link, child back_left_standoff_link, origin xyz=-0.048 0.008 0.029 rpy=0.0 0.0 0.0
- added joint bottom_tail_to_back_right_standoff_joint: type fixed, parent bottom_tail_link, child back_right_standoff_link, origin xyz=-0.048 -0.008 0.029 rpy=0.0 0.0 0.0
- added joint bottom_tail_to_front_left_standoff_joint: type fixed, parent bottom_tail_link, child front_left_standoff_link, origin xyz=0.048 0.008 0.029 rpy=0.0 0.0 0.0
- added joint bottom_tail_to_front_right_standoff_joint: type fixed, parent bottom_tail_link, child front_right_standoff_link, origin xyz=0.048 -0.008 0.029 rpy=0.0 0.0 0.0
- added joint bottom_tail_to_tail_bracket_joint: type fixed, parent tail_bracket, child bottom_tail_link, origin xyz=-0.078 0.0 0.005 rpy=0.0 0.0 0.0
- added joint camera_board_to_camera_bracket_joint: type fixed, parent camera_mount_bracket_2_link, child camera_board_link, origin xyz=0.002 0.0 0.0 rpy=0.0 0.0 0.0
- added joint camera_board_to_camera_lens_joint: type fixed, parent camera_board_link, child camera_lens_link, origin xyz=0.009 0.0 -0.0035 rpy=1.5708 3.1416 1.5708
- added joint castor_to_castor_wheel_joint: type continuous, parent castor_link, child castor_wheel_link, origin xyz=0.0 0.0 -0.013 rpy=-1.5708 0 0, axis 0 0 1
- added joint imu_to_imu_left_standoff_joint: type fixed, parent imu_link, child imu_left_standoff_link, origin xyz=0.0108 0.0076 -0.011 rpy=0.0 0.0 0.0
- added joint imu_to_imu_right_standoff_joint: type fixed, parent imu_link, child imu_right_standoff_link, origin xyz=0.0108 -0.0076 -0.011 rpy=0.0 0.0 0.0
- added joint leddar_sensor_to_front_base_plate_joint: type fixed, parent base_link, child leddar_sensor_link, origin xyz=0.01045 0.0 0.062 rpy=0.0 0.0 0.0
- added joint leddar_sensor_to_led_lens_joint: type fixed, parent leddar_sensor_link, child leddar_lens_link, origin xyz=0.0165 -0.014 0.023 rpy=1.5708 3.1416 1.5708
- added joint left_motor_bracket_to_left_motor_joint: type fixed, parent left_motor_bracket_link, child left_motor_link, origin xyz=0.0  -0.03325 -0.006 rpy=-1.5708 0.0 0.0
- added joint left_motor_output_to_left_wheel_connector_joint: type fixed, parent left_motor_output_shaft_link, child left_wheel_connector_link, origin xyz=0.0 0.0 0.0 rpy=0.0 0.0 0.0
- added joint left_motor_to_left_motor_output_shaft_joint: type continuous, parent left_motor_link, child left_motor_output_shaft_link, origin xyz=0.0 0.0 0.038 rpy=0.0 0.0 0.0, axis 0 0 1
- added joint left_wheel_connector_to_left_wheel_joint: type fixed, parent left_wheel_connector_link, child left_wheel_link, origin xyz=0.0 0.0 0.00625 rpy=0.0 0.0 0.0
- added joint right_motor_bracket_to_right_motor_joint: type fixed, parent right_motor_bracket_link, child right_motor_link, origin xyz=0.0  0.03325 -0.006 rpy=1.5708 0.0 0.0
- added joint right_motor_output_to_right_wheel_connector_joint: type fixed, parent right_motor_output_shaft_link, child right_wheel_connector_link, origin xyz=0.0 0.0 0.0 rpy=0.0 0.0 0.0
- added joint right_motor_to_right_motor_output_shaft_joint: type continuous, parent right_motor_link, child right_motor_output_shaft_link, origin xyz=0.0 0.0 0.038 rpy=0.0 0.0 0.0, axis 0 0 1
- added joint right_wheel_connector_to_right_wheel_joint: type fixed, parent right_wheel_connector_link, child right_wheel_link, origin xyz=0.0 0.0 0.00625 rpy=0.0 0.0 0.0
- added joint tail_base_plate_to_raspberry_p_plate: type fixed, parent tail_base_plate_link, child raspberry_pi_link, origin xyz=0.0 0.0085 0.018 rpy=0.0 0.0 0.0
- added joint top_tail_to_bottom_tail_joint: type fixed, parent bottom_tail_link, child top_tail_link, origin xyz=0.008 0.0 0.054 rpy=0.0 0.0 0.0
- added joint top_tail_to_tail_base_plate_joint: type fixed, parent top_tail_link, child tail_base_plate_link, origin xyz=-0.017 0.0 0.0055 rpy=0.0 0.0 0.0
- joint angle_bracket_joint: child angle_bracket_plate_2 -> angle_bracket_plate_2_link; origin xyz=0.012 0.0 0.013 rpy=0.0 1.5708 0.0 -> xyz=0.012 0.0 0.013 rpy=0.0 0.0 0.0; parent angle_bracket_plate_1 -> angle_bracket_plate_1_link
- joint base_to_left_motor_bracket_joint: child left_motor_bracket -> left_motor_bracket_link; origin xyz=-0.0735 0.0 -0.0145 rpy=0.0 -1.5708 0.0 -> xyz=0.0 0.0735 -0.0145 rpy=0.0 0.0 0.0
- joint base_to_right_motor_bracket_joint: child right_motor_bracket -> right_motor_bracket_link; origin xyz=0.0735 0.0 -0.0145 rpy=0.0 -1.5708 0.0 -> xyz=0.0 -0.0735 -0.0145 rpy=0.0 0.0 0.0
- joint base_to_tail_bracket_joint: origin xyz=0.0 -0.012 -0.005 rpy=0.0 0.0 1.5707 -> xyz=-0.012 0.0 -0.005 rpy=0.0 0.0 0.0
- joint camera_mount_bracket_joint: child camera_mount_bracket_2 -> camera_mount_bracket_2_link; origin xyz=0.0 0.010 -0.0025 rpy=0.0 0.0 0.0 -> xyz=0.010 0.0 -0.0025 rpy=0.0 0.0 0.0; parent camera_mount_bracket_1 -> camera_mount_bracket_1_link
- joint camera_mount_to_leddar_sensor_joint: child camera_mount_bracket_1 -> camera_mount_bracket_1_link; origin xyz=0.0 0.02045 0.0595 rpy=0.0 0.0 0.0 -> xyz=0.02045 0.0 0.0595 rpy=0.0 0.0 0.0; parent leddar_sensor -> leddar_sensor_link
- joint castor_joint: child castor -> castor_link; parent castor_bracket -> castor_bracket_link
- joint imu_to_top_tail_link_joint: child imu -> imu_link; origin xyz=0.0427 0.0 0.025 rpy=0.0 0.0 -1.5708 -> xyz=0.0427 0.0 0.025 rpy=0.0 0.0 0.0
- joint tail_to_castor_bracket_joint: child castor_bracket -> castor_bracket_link; parent tail_link -> bottom_tail_link
